File: src/main/kicad/kicad-weird-board-fp/kicad-weird-board-fp.sch (KiCad schematic (older format))
At the start: 49 parts

Commit message: Kicad WIP board
Parts:
- added U?: MCP23017_SP, Package_DIP:DIP-28_W7.62mm, symbol Interface_Expansion:MCP23017_SP
Changed lines of the file:
@@
 	0    -1   -1   0
 $EndComp
+$Comp
+L Interface_Expansion:MCP23017_SP U?
+U 1 1 65E1C25D
+P 2300 4800
+F 0 "U?" H 2300 6081 50  0000 C CNN
+F 1 "MCP23017_SP" H 2300 5990 50  0000 C CNN
+F 2 "Package_DIP:DIP-28_W7.62mm" H 2500 3800 50  0001 L CNN
+F 3 "http://ww1.microchip.com/downloads/en/DeviceDoc/20001952C.pdf" H 2500 3700 50  0001 L CNN
+	1    2300 4800
+	1    0    0    -1
+$EndComp
 $EndSCHEMATC

Commit message: Kicad WIP board
Parts:
- added C1: 100nF, symbol Device:C
- added RSCL, RSDA: 4.7k, symbol Device:R
- JFP: value Screw_Terminal_01x08 -> ST 1x8
- gave numbers to parts that had none: 1
Connections:
- net +3V3: now also IOE.9 (VDD), C1.2, RSCL.2, RSDA.2
- net at R1A.1: now also IOE.1 (GPB0)
- net at R1B.2: now also IOE.2 (GPB1)
- net at R2A.2: now also IOE.3 (GPB2)
- net at R2B.2: now also IOE.4 (GPB3)
- net at R3A.2: now also IOE.5 (GPB4)
- net at R3B.2: now also IOE.6 (GPB5)
- net at R4A.2: now also IOE.7 (GPB6)
- net at R4B.2: now also IOE.8 (GPB7)
- net at R5A.2: now also IOE.21 (GPA0)
- net at R5B.2: now also IOE.22 (GPA1)
- net at R6A.2: now also IOE.23 (GPA2)
- net at R6B.2: now also IOE.24 (GPA3)
- net at R7A.2: now also IOE.25 (GPA4)
- net at R7B.2: now also IOE.26 (GPA5)
- net at R8A.2: now also IOE.27 (GPA6)
- net at R8B.2: now also IOE.28 (GPA7)
- net GNDD: now reaches IOE.10 (VSS)
- net GNDD: now also IOE.15 (A0), IOE.16 (A1), IOE.17 (A2), C1.1
- net SCL: now reaches IOE.12 (SCK)
- net SCL: now also RSCL.1
- net SDA: now reaches IOE.13 (SDA)
- net SDA: now also RSDA.1
Other:
- moved on the sheet: D1A, D1B, D2A, D2B, D3A, D3B, D4A, D4B, D5A, D5B, D6A, D6B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
